File: hardware/Typhoon Motherboard KiCad.kicad_sch (KiCad schematic)
At the start: 45 parts, among them J1 Conn_01x04_Pin, J2 Conn_02x03_Odd_Even, P1 USB_C_Plug_USB2.0, U1 ESP32-S3-WROOM-1, U2 TPS54360DDA, U3 TJA1051T-3, U7 MCP1825S

Commit message: added to do list in the schematic notes lol
Other:
- note added: "still to do: - add uart conenction for telemetry - add power out connections for peripheral boards when in wired power operation mode"
- moved on the sheet: BT1
Changed lines of the file:
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@@
 	)
 	(junction
-		(at 194.31 45.72)
+		(at 194.31 33.02)
 		(diameter 0)
 		(color 0 0 0 0)
 	)
 	(junction
-		(at 194.31 55.88)
+		(at 194.31 43.18)
 		(diameter 0)
 		(color 0 0 0 0)
@@
 	(wire
 		(pts
-			(xy 189.23 60.96) (xy 189.23 55.88)
+			(xy 189.23 48.26) (xy 189.23 43.18)
 		)
 		(stroke
@@
 	(wire
 		(pts
-			(xy 199.39 60.96) (xy 199.39 55.88)
+			(xy 199.39 48.26) (xy 199.39 43.18)
 		)
 		(stroke
@@
 	(wire
 		(pts
-			(xy 194.31 55.88) (xy 194.31 54.61)
+			(xy 194.31 43.18) (xy 194.31 41.91)
 		)
 		(stroke
@@
 	(wire
 		(pts
-			(xy 199.39 55.88) (xy 194.31 55.88)
+			(xy 199.39 43.18) (xy 194.31 43.18)
 		)
 		(stroke
@@
 	(wire
 		(pts
-			(xy 189.23 45.72) (xy 194.31 45.72)
+			(xy 189.23 33.02) (xy 194.31 33.02)
 		)
 		(stroke
@@
 	(wire
 		(pts
-			(xy 199.39 40.64) (xy 199.39 45.72)
+			(xy 199.39 27.94) (xy 199.39 33.02)
 		)
 		(stroke
@@
 	(wire
 		(pts
-			(xy 189.23 40.64) (xy 189.23 45.72)
+			(xy 189.23 27.94) (xy 189.23 33.02)
 		)
 		(stroke
@@
 	(wire
 		(pts
-			(xy 194.31 45.72) (xy 194.31 46.99)
+			(xy 194.31 33.02) (xy 194.31 34.29)
 		)
 		(stroke
@@
 	(wire
 		(pts
-			(xy 199.39 45.72) (xy 194.31 45.72)
+			(xy 199.39 33.02) (xy 194.31 33.02)
 		)
 		(stroke
@@
 	(wire
 		(pts
-			(xy 189.23 55.88) (xy 194.31 55.88)
+			(xy 189.23 43.18) (xy 194.31 43.18)
 		)
 		(stroke
@@
 	)
 	(rectangle
-		(start 182.88 30.48)
-		(end 212.09 76.2)
+		(start 182.88 17.78)
+		(end 212.09 63.5)
 		(stroke
 			(width 0)
@@
 		)
 	)
+	(text "still to do:\n\n- add uart conenction\nfor telemetry\n\n- add power out connections\nfor peripheral boards when\nin wired power operation mode"
+		(exclude_from_sim no)
+		(at 180.848 78.74 0)
+		(effects
+			(font
+				(size 1.27 1.27)
+			)
+			(justify left)
+		)
+	)
 	(text "Battery Connection\n(3.7V-5V, XT30)"
 		(exclude_from_sim no)
-		(at 184.15 72.898 0)
+		(at 184.15 60.198 0)
 		(effects
 			(font
@@
 	(symbol
 		(lib_id "power:+BATT")
-		(at 189.23 40.64 0)
+		(at 189.23 27.94 0)
 		(unit 1)
 		(exclude_from_sim no)
@@
 		(dnp no)
 		(property "Reference" "#PWR015"
-			(at 189.23 44.45 0)
+			(at 189.23 31.75 0)
 			(effects
 				(font
@@
 		)
 		(property "Value" "+BATT"
-			(at 189.23 35.56 0)
+			(at 189.23 22.86 0)
 			(effects
 				(font
@@
 		)
 		(property "Footprint" ""
-			(at 189.23 40.64 0)
+			(at 189.23 27.94 0)
 			(effects
 				(font
@@
 		)
 		(property "Datasheet" ""
-			(at 189.23 40.64 0)
+			(at 189.23 27.94 0)
 			(effects
 				(font
@@
 		)
 		(property "Description" "Power symbol creates a global label with name \"+BATT\""
-			(at 189.23 40.64 0)
+			(at 189.23 27.94 0)
 			(effects
 				(font
@@
 	(symbol
 		(lib_id "power:GND")
-		(at 199.39 60.96 0)
+		(at 199.39 48.26 0)
 		(unit 1)
 		(exclude_from_sim no)
@@
 		(fields_autoplaced yes)
 		(property "Reference" "#PWR027"
-			(at 199.39 67.31 0)
+			(at 199.39 54.61 0)
 			(effects
 				(font
@@
 		)
 		(property "Value" "GND"
-			(at 199.39 66.04 0)
+			(at 199.39 53.34 0)
 			(effects
 				(font
@@
 		)
 		(property "Footprint" ""
-			(at 199.39 60.96 0)
+			(at 199.39 48.26 0)
 			(effects
 				(font
@@
 		)
 		(property "Datasheet" ""
-			(at 199.39 60.96 0)
+			(at 199.39 48.26 0)
 			(effects
 				(font
@@
 		)
 		(property "Description" "Power symbol creates a global label with name \"GND\" , ground"
-			(at 199.39 60.96 0)
+			(at 199.39 48.26 0)
 			(effects
 				(font
@@
 	(symbol
 		(lib_id "power:-BATT")
-		(at 189.23 60.96 180)
+		(at 189.23 48.26 180)
 		(unit 1)
 		(exclude_from_sim no)
@@
 		(fields_autoplaced yes)
 		(property "Reference" "#PWR025"
-			(at 189.23 57.15 0)
+			(at 189.23 44.45 0)
 			(effects
 				(font
@@
 		)
 		(property "Value" "-BATT"
-			(at 189.23 66.04 0)
+			(at 189.23 53.34 0)
 			(effects
 				(font
@@
 		)
 		(property "Footprint" ""
-			(at 189.23 60.96 0)
+			(at 189.23 48.26 0)
 			(effects
 				(font
@@
 		)
 		(property "Datasheet" ""
-			(at 189.23 60.96 0)
+			(at 189.23 48.26 0)
 			(effects
 				(font
@@
 		)
 		(property "Description" "Power symbol creates a global label with name \"-BATT\""
-			(at 189.23 60.96 0)
+			(at 189.23 48.26 0)
 			(effects
 				(font
@@
 	(symbol
 		(lib_id "power:+5V")
-		(at 199.39 40.64 0)
+		(at 199.39 27.94 0)
 		(unit 1)
 		(exclude_from_sim no)
@@
 		(fields_autoplaced yes)
 		(property "Reference" "#PWR042"
-			(at 199.39 44.45 0)
+			(at 199.39 31.75 0)
 			(effects
 				(font
@@
 		)
 		(property "Value" "+5V"
-			(at 199.39 35.56 0)
+			(at 199.39 22.86 0)
 			(effects
 				(font
@@
 		)
 		(property "Footprint" ""
-			(at 199.39 40.64 0)
+			(at 199.39 27.94 0)
 			(effects
 				(font
@@
 		)
 		(property "Datasheet" ""
-			(at 199.39 40.64 0)
+			(at 199.39 27.94 0)
 			(effects
 				(font
@@
 		)
 		(property "Description" "Power symbol creates a global label with name \"+5V\""
-			(at 199.39 40.64 0)
+			(at 199.39 27.94 0)
 			(effects
 				(font
@@
 	(symbol
 		(lib_id "Device:Battery_Cell")
-		(at 194.31 52.07 0)
+		(at 194.31 39.37 0)
 		(unit 1)
 		(exclude_from_sim no)
@@
 		(fields_autoplaced yes)
 		(property "Reference" "BT1"
-			(at 198.12 48.9584 0)
+			(at 198.12 36.2584 0)
 			(effects
 				(font
@@
 		)
 		(property "Value" "Battery_Cell"
-			(at 198.12 51.4984 0)
+			(at 198.12 38.7984 0)
 			(effects
 				(font
@@
 		)
 		(property "Footprint" "Connector_AMASS:AMASS_XT30PW-M_1x02_P2.50mm_Horizontal"
-			(at 194.31 50.546 90)
+			(at 194.31 37.846 90)
 			(effects
 				(font
@@
 		)
 		(property "Datasheet" "~"
-			(at 194.31 50.546 90)
+			(at 194.31 37.846 90)
 			(effects
 				(font
@@
 		)
 		(property "Description" "Single-cell battery"
-			(at 194.31 52.07 0)
+			(at 194.31 39.37 0)
 			(effects
 				(font
