File: hardware/CentralPowerSource.kicad_sch (KiCad schematic)
At the start: 23 parts, among them J11 Conn_01x02_Pin, J12 Conn_01x02_Pin, J13 Conn_01x02_Pin, J14 Conn_01x02_Pin, J15 Conn_01x02_Pin, J16 Conn_01x02_Pin, U4 TPS54331DDA

Commit message: Updated the Boost Converter
Parts:
- removed C16, C22: 4.7u, Capacitor_SMD:C_0603_1608Metric, symbol Device:C
- removed C23: 0.1u, Capacitor_SMD:C_0603_1608Metric, symbol Device:C
- removed C24: 0.01u, Capacitor_SMD:C_0603_1608Metric, symbol Device:C
- removed C25: 1000p, Capacitor_SMD:C_0603_1608Metric, symbol Device:C
- removed C26, C27, C28: 47u, Capacitor_SMD:C_0603_1608Metric, symbol Device:C
- removed D5: B340, Diode_SMD:D_SMC, symbol Diode:B340
- removed L2: 4.7u, Inductor_SMD:L_Taiyo-Yuden_NR-60xx, symbol Device:L
- removed R17: 29.4k, Resistor_SMD:R_0603_1608Metric, symbol Device:R
- removed R18: 10.2k, Resistor_SMD:R_0603_1608Metric, symbol Device:R
- removed R19: 3.24k, Resistor_SMD:R_0603_1608Metric, symbol Device:R
- removed U4: TPS54331DDA, Package_SO:TI_SO-PowerPAD-8_ThermalVias, symbol Regulator_Switching:TPS54360DDA
- added C11: 0.1 uF, Capacitor_SMD:C_0603_1608Metric, symbol Device:C
- added C7: 20uF, Capacitor_SMD:C_0603_1608Metric, symbol Device:C
- added C9: 66uF, Capacitor_SMD:C_0603_1608Metric, symbol Device:C
- added D5: LED, LED_SMD:LED_0805_2012Metric, symbol Device:LED
- added L1: 1 uH, Inductor_SMD:L_0805_2012Metric, symbol Device:L
- added R5: 1M, Resistor_SMD:R_0603_1608Metric, symbol Device:R
- added R6: 111k, Resistor_SMD:R_0603_1608Metric, symbol Device:R
- added U3: TPS63060, Package_SON:Texas_S-PWSON-N10_ThermalVias, symbol Regulator_Switching:TPS63060
- C10: value 4.7u -> 10pF
- R15: value 200k -> 1M
- R16: value 98k -> 330
Connections:
- net +BATT: now also C7.1, U3.2 (VIN), U3.3 (EN); no longer C10.1, R15.1
- net GND: now also C11.1, C7.2, C9.2, D5.1 (K), R6.2, U3.11 (PGND), U3.4 (PS/SYNC), U3.7 (GND); no longer R16.2
- net PG: now reaches R15.2, R16.1
- net PG: now also U3.5 (PG)
- net +3.3VA renamed +5VA
- net +5VA: now also R15.1, C9.1, R5.1, U3.9 (VOUT)
- new net: L1.1, U3.1 (L1)
- new net: L1.2, U3.10 (L2)
- new net: C11.2, U3.6 (VAUX)
- new net: C10.1, R5.2, R6.1, U3.8 (FB)
- new net: D5.2 (A), R16.2
- no-connect marks 1 -> 0
Other:
- note added: "Batt -> 5V boost converter"
- note added: "LED on if power good"
- note removed: "3.7V-5V Regulator (for use when TYPHOON is operating in central power source configuration, and MOTHERBOARD is operating as a power distributor)"

Commit message: Production Files
Connections:
- net +BATT: no longer C7.1
- net GND: no longer C7.2
Other:
- moved on the sheet: C7
Changed lines of the file:
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@@
-	)
-	(junction
-		(at 128.27 85.09)
-		(diameter 0)
-		(color 0 0 0 0)
 	)
 	(junction
@@
 	(junction
 		(at 101.6 109.22)
-		(diameter 0)
-		(color 0 0 0 0)
-	)
-	(junction
-		(at 128.27 77.47)
 		(diameter 0)
 		(color 0 0 0 0)
@@
 	(symbol
 		(lib_id "Device:C")
-		(at 128.27 81.28 0)
+		(at 128.27 81.28 90)
 		(unit 1)
 		(exclude_from_sim no)
@@
 		(fields_autoplaced yes)
 		(property "Reference" "C7"
-			(at 132.08 80.0099 0)
-			(effects
-				(font
-					(size 1.27 1.27)
-				)
-				(justify left)
+			(at 128.27 73.66 90)
+			(effects
+				(font
+					(size 1.27 1.27)
+				)
 			)
 		)
 		(property "Value" "20uF"
-			(at 132.08 82.5499 0)
-			(effects
-				(font
-					(size 1.27 1.27)
-				)
-				(justify left)
+			(at 128.27 76.2 90)
+			(effects
+				(font
+					(size 1.27 1.27)
+				)
 			)
 		)
 		(property "Footprint" "Capacitor_SMD:C_0603_1608Metric"
-			(at 129.2352 85.09 0)
-			(effects
-				(font
+			(at 132.08 80.3148 0)
+			(effects
+				(font
