File: hardware/rev0/CentralPowerSource.kicad_sch (KiCad schematic)
At the start: 17 parts, among them J11 Conn_01x02_Pin, J12 Conn_01x02_Pin, J13 Conn_01x02_Pin, J14 Conn_01x02_Pin, J15 Conn_01x02_Pin, J16 Conn_01x02_Pin, U3 TPS63060

Commit message: Updated Rev 1
Parts:
- removed J15, J16: Conn_01x02_Pin, Connector_PinHeader_2.00mm:PinHeader_1x02_P2.00mm_Vertical_SMD_Pin1Right, symbol Connector:Conn_01x02_Pin
- J11, J12, J13, J14: footprint Connector_PinHeader_2.00mm:PinHeader_1x02_P2.00mm_Vertical_SMD_Pin1Right -> Connector_JST:JST_EH_S2B-EH_1x02_P2.50mm_Horizontal
