File: hardware/rev0/Typhoon Motherboard KiCad.kicad_pcb (KiCad board)
At the start: 2 copper layers, 73.5 x 52.8 mm, 55 parts, among them J1 Conn_01x04_Pin, J10 USB_C_Receptacle_USB2.0, J11 Conn_01x02_Pin, J12 Conn_01x02_Pin, J13 Conn_01x02_Pin, J14 Conn_01x02_Pin, J15 Conn_01x02_Pin, J16 Conn_01x02_Pin, J2 Conn_02x03_Odd_Even, J3 Conn_01x04_Pin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

Commit message: Updated Rev 1
Parts:
- J1: footprint Connector_PinHeader_2.00mm:PinHeader_1x04_P2.00mm_Vertical -> Connector_JST:JST_EH_S4B-EH_1x04_P2.50mm_Horizontal
- J11, J12, J13, J14: footprint Connector_PinHeader_2.00mm:PinHeader_1x02_P2.00mm_Vertical_SMD_Pin1Right -> Connector_JST:JST_EH_S2B-EH_1x02_P2.50mm_Horizontal
Connections:
- J10 pad A6: /D+ -> Net-(J10-D+-PadA6)
- J10 pad A7: /D- -> Net-(J10-D--PadA7)
- J10 pad B6: /D+ -> Net-(J10-D+-PadA6)
- J10 pad B7: /D- -> Net-(J10-D--PadA7)
- R1 pad 2: /D- -> Net-(J10-D--PadA7)
- R2 pad 2: /D+ -> Net-(J10-D+-PadA6)
Routing:
- net /D-: track 29.1 -> 22.7 mm
- net Net-(J10-D--PadA7): track 0.00 -> 5.97 mm
Other:
- board text added: "TYPHOON MOTHERBOARD VERSION 1"
