File: hardware/rev0/Typhoon Motherboard KiCad.kicad_sch (KiCad schematic)
At the start: 38 parts, among them J1 Conn_01x04_Pin, J10 USB_C_Receptacle_USB2.0, J2 Conn_02x03_Odd_Even, J3 Conn_01x04_Pin, U1 ESP32-S3-WROOM-1, U2 SN65HVD233, U7 MCP1825S

Commit message: Updated Rev 1
Parts:
- J1: footprint Connector_PinHeader_2.00mm:PinHeader_1x04_P2.00mm_Vertical -> Connector_JST:JST_EH_S4B-EH_1x04_P2.50mm_Horizontal
Changed lines of the file:
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@@
 			)
 		)
-		(property "Footprint" "Connector_PinHeader_2.00mm:PinHeader_1x04_P2.00mm_Vertical"
+		(property "Footprint" "Connector_JST:JST_EH_S4B-EH_1x04_P2.50mm_Horizontal"
 			(at 246.38 30.48 0)
 			(effects
