File: hardware/rev2/TyphoonMotherboard_rev1 KiCad.kicad_pcb (KiCad board)
At the start: 2 copper layers, 55.9 x 49.5 mm, 75 parts, among them J1 Conn_02x04_Odd_Even, J2 Conn_01x04_Pin, J3 UJ20-C-H-C-4-SMT-TR, J5 Conn_01x02_Pin, J6 Conn_01x02_Pin, J7 Conn_01x04_Pin, SW1 SW_Push, SW2 SW_Push, SW3 SW_Push, U1 USBLC6-2SC6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

Commit message: removed updates
Parts:
- removed C1: 1uF, Capacitor_SMD:C_0603_1608Metric
- removed C10: 47uF, Capacitor_SMD:C_0603_1608Metric
- removed C11: 47nF, Capacitor_SMD:C_0603_1608Metric
- removed C12: 4.7uF, Capacitor_SMD:C_0603_1608Metric
- removed C13, C14, C3, C8, C9: 10uF, Capacitor_SMD:C_0603_1608Metric
- removed C16, C17: 22uF, Capacitor_SMD:C_0603_1608Metric
- removed D1, D5, D6: LED, LED_SMD:LED_0805_2012Metric
- removed D8: SMBJ5.0A, SMBJ5.0A:DIOM4336X265N
- removed J3: UJ20-C-H-C-4-SMT-TR, UJ20-C-H-C-4-SMT-TR:CUI_UJ20-C-H-C-4-SMT-TR
- removed L1: 2.2uH, Inductor_SMD:L_0805_2012Metric
- removed L2, L3: 0.47uH, Inductor_SMD:L_0603_1608Metric
- removed R1, R11, R17, R18, R2: 10k, Resistor_SMD:R_0603_1608Metric
- removed R10, R9: 320, Resistor_SMD:R_0603_1608Metric
- removed R19: 280, Resistor_SMD:R_0603_1608Metric
- removed R20: 330, Resistor_SMD:R_0603_1608Metric
- removed R21: 511k, Resistor_SMD:R_0603_1608Metric
- removed R24: 5.23k, Resistor_SMD:R_0603_1608Metric
- removed R25, R29: 91k, Resistor_SMD:R_0603_1608Metric
- removed R26, R27: 100k, Resistor_SMD:R_0603_1608Metric
- removed R28: 806k, Resistor_SMD:R_0603_1608Metric
- removed RT1: 103AT-2, 103AT-2:103AT-2
- removed U6: TPS63802DLAR, TPS63802DLAR (1):VREG_TPS63802DLAR
- C5: value 10u -> 10uF
- U4: value BQ25895RTW -> TPS62130A; footprint Package_DFN_QFN:Texas_RTW_WQFN-24-1EP_4x4mm_P0.5mm_EP2.7x2.7mm_ThermalVias -> Package_DFN_QFN:VQFN-16-1EP_3x3mm_P0.5mm_EP1.68x1.68mm_ThermalVias
- U5: value TPS63802DLAR -> TPS62130A; footprint TPS63802DLAR (1):VREG_TPS63802DLAR -> Package_DFN_QFN:VQFN-16-1EP_3x3mm_P0.5mm_EP1.68x1.68mm_ThermalVias
- moved SW2 97.0 mm to (162.3, 71.6), turned to 0 degrees
- moved U1 86.8 mm to (155.5, 102.9)
- moved R14 85.6 mm to (146.9, 98.7), turned to 0 degrees
- moved R8 82.0 mm to (146.9, 91.2), turned to 0 degrees
- moved R22 79.1 mm to (150.9, 93.7)
- moved R7 78.9 mm to (146.9, 88.7), turned to 0 degrees
- moved C18 77.5 mm to (142.9, 98.7), turned to 0 degrees
- moved C5 77.1 mm to (142.9, 91.2), turned to 0 degrees
- moved R12 77.0 mm to (146.9, 93.7)
- moved U3 75.3 mm to (166.6, 100.5), turned to 0 degrees
- moved H1 73.0 mm to (129.7, 95.3)
- moved D4 72.1 mm to (136.2, 101.7), turned to 0 degrees
- moved C2 71.4 mm to (142.9, 86.2), turned to 0 degrees
- moved H3 71.3 mm to (137.4, 86.7)
- moved G*** 70.4 mm to (147.8, 108.2)
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Connections:
- C15 pad 2: +3.3V -> +3v3
- C18 pad 1: V_{USB-C} -> V_USB-C
- C2 pad 1: +3.3V -> +3V3
- C4 pad 1: +3.3V -> +3V3
- C5 pad 1: +3.3V -> +3V3
- D10 pad 2: +3.3V -> +3V3
- J2 pad 2: +3.3V -> +3V3
- U2 pad 12: /LED_{4} -> unconnected-(U2-IO8-Pad12)
- U2 pad 19: /PMIC_{SDA} -> unconnected-(U2-IO11-Pad19)
- U2 pad 2: +3.3V -> +3V3
- U2 pad 20: /PMIC_{SCL} -> unconnected-(U2-IO12-Pad20)
- U2 pad 21: /PMIC_{NQON} -> unconnected-(U2-IO13-Pad21)
- U2 pad 22: /PMIC_{INT} -> unconnected-(U2-IO14-Pad22)
- U2 pad 7: /LED_{3} -> unconnected-(U2-IO7-Pad7)
- U2 pad 8: /PMIC_{OTG} -> unconnected-(U2-IO15-Pad8)
- U2 pad 9: /PMIC_{CE} -> unconnected-(U2-IO16-Pad9)
- U3 pad 3: +3.3V -> +3v3
- U4 pad 1: V_{USB-C} -> Net-(L1-Pad1)
- U4 pad 10: Net-(U4-ILIM) -> +6.2V
- U4 pad 11: Net-(U4-TS) -> +6.2V
- U4 pad 12: /PMIC_{NQON} -> +6.2V
- U4 pad 13: +BATT -> +6.2V
- U4 pad 14: +BATT -> +5V
- U4 pad 15: V_{SYS} -> Net-(U4-GND-Pad15)
- U4 pad 16: V_{SYS} -> Net-(U4-GND-Pad15)
- U4 pad 17: GND -> Net-(U4-GND-Pad15)
- U4 pad 2: unconnected-(U4-D+-Pad2) -> Net-(L1-Pad1)
- U4 pad 3: unconnected-(U4-D--Pad3) -> Net-(L1-Pad1)
- U4 pad 4: Net-(U4-STAT) -> unconnected-(U4-PG-Pad4)
- U4 pad 5: /PMIC_{SCL} -> unconnected-(U4-FB-Pad5)
- U4 pad 6: /PMIC_{SDA} -> Net-(U4-GND-Pad15)
- U4 pad 7: /PMIC_{INT} -> unconnected-(U4-FSW-Pad7)
- U4 pad 8: /PMIC_{OTG} -> unconnected-(U4-DEF-Pad8)
- U4 pad 9: /PMIC_{CE} -> unconnected-(U4-SS/TR-Pad9)
- U5 pad 1: V_{SYS} -> Net-(L2-Pad1)
- U5 pad 10: V_{SYS} -> +6.2V
- U5 pad 2: GND -> Net-(L2-Pad1)
- U5 pad 3: GND -> Net-(L2-Pad1)
- U5 pad 4: Net-(U5-FB) -> unconnected-(U5-PG-Pad4)
- U5 pad 5: Net-(U5-PG) -> unconnected-(U5-FB-Pad5)
- U5 pad 6: +3.3V -> Net-(U5-GND-Pad15)
- U5 pad 7: Net-(U5-L2) -> unconnected-(U5-FSW-Pad7)
- U5 pad 8: GND -> unconnected-(U5-DEF-Pad8)
- U5 pad 9: Net-(U5-L1) -> unconnected-(U5-SS/TR-Pad9)
Routing:
- net +5V: track 71.0 -> 0.00 mm
- net V_{USB-C}: track 60.1 -> 0.00 mm, vias 2 -> 0
- net V_{SYS}: track 44.0 -> 0.00 mm, vias 2 -> 0
- net /LED_{2}: track 35.3 -> 0.00 mm, vias 2 -> 0
- net /LED_{1}: track 33.9 -> 0.00 mm, vias 2 -> 0
- net /GPIO_{3}: track 33.9 -> 0.00 mm
- net /GPIO_{4}: track 33.1 -> 0.00 mm
- net +BATT: track 32.4 -> 0.00 mm
- net /PMIC_{OTG}: track 31.2 -> 0.00 mm, vias 3 -> 0
- net /GPIO_{6}: track 30.1 -> 0.00 mm, vias 1 -> 0
- net /Mother_{RX}: track 43.2 -> 15.1 mm, vias 1 -> 0
- net GND: track 27.6 -> 0.00 mm, vias 35 -> 0
- net /GPIO_{2}: track 27.1 -> 0.00 mm
- net /EN: track 26.8 -> 0.00 mm
- net /LED_{3}: track 26.7 -> 0.00 mm, vias 2 -> 0
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- added copper zone on F.Cu, net +5V
- removed copper zone on F.Cu, net +3.3V
Other:
- board size 55.9 x 49.5 mm -> 60.4 x 48.6 mm
- board text removed: "3.3V"
- board text removed: "3.3V REG"
- board text removed: "5V"
- board text removed: "5V REG"
- board text removed: "BMIC"
- board text removed: "Battery Conn."
- board text removed: "CAN TRAN."
- board text removed: "CAN+"
- board text removed: "CAN-"
- board text removed: "EN"
- board text removed: "GND"
- board text removed: "J. Lo"
- board text removed: "LED_{1}"
- board text removed: "LED_{2}"
- board text removed: "LED_{3}"
- board text removed: "LED_{4}"
- board text removed: "RX"
- board text removed: "STATUS LED"
- board text removed: "TX"
- board text removed: "TYPHOON MOTHERBOARD"
- board text removed: "V2.0"

Commit message: some other small changes
Parts:
- removed BT1: XT30, Connector_AMASS:AMASS_XT30U-F_1x02_P5.0mm_Vertical
- removed C18: 10uF, Capacitor_SMD:C_0603_1608Metric
- removed G***: LOGO, hpvdt-log.preety:hpvdt-logo
- removed U5: TPS62130A, Package_DFN_QFN:VQFN-16-1EP_3x3mm_P0.5mm_EP1.68x1.68mm_ThermalVias
- added C1: 10uF, Capacitor_SMD:C_0603_1608Metric, F.Cu at (164.9, 79.3)
- added C10: 3.3nF, Capacitor_SMD:C_0603_1608Metric, F.Cu at (168.9, 84.3)
- added C11: 0.1uF, Capacitor_SMD:C_0603_1608Metric, F.Cu at (168.9, 86.8)
- added C12: 0.1uF, Capacitor_SMD:C_0603_1608Metric, F.Cu at (168.9, 89.3)
- added C3: 22uF, Capacitor_SMD:C_0603_1608Metric, F.Cu at (164.9, 84.3)
- added C7: 10uF, Capacitor_SMD:C_0603_1608Metric, F.Cu at (164.9, 94.3)
- added C8: 22uF, Capacitor_SMD:C_0603_1608Metric, F.Cu at (168.9, 79.3)
- added C9: 3.3nF, Capacitor_SMD:C_0603_1608Metric, F.Cu at (168.9, 81.8)
- added F1: Polyfuse, Fuse:Fuse_1206_3216Metric, F.Cu at (151.2, 103.1)
- added J10: USB_C_Receptacle_USB2.0_16P, Connector_USB:USB_C_Receptacle_JAE_DX07S016JA1R1500, F.Cu at (183.4, 101.8)
- added J11: Conn_01x02_Pin, Connector_JST:JST_XH_B2B-XH-A_1x02_P2.50mm_Vertical, F.Cu at (135.5, 112.6)
- added J4: Conn_01x04_Pin, Connector_JST:JST_XH_B4B-XH-A_1x04_P2.50mm_Vertical, F.Cu at (151.9, 89.2)
- added J8: Conn_01x02_Pin, Connector_JST:JST_XH_B2B-XH-A_1x02_P2.50mm_Vertical, F.Cu at (135.5, 97.0)
- added J9: Conn_01x02_Pin, Connector_JST:JST_XH_B2B-XH-A_1x02_P2.50mm_Vertical, F.Cu at (135.5, 104.8)
- added L1: 2.2uH, Inductor_SMD:L_0805_2012Metric, F.Cu at (143.7, 116.3)
- added L2: 2.2uH, Inductor_SMD:L_0805_2012Metric, F.Cu at (143.7, 119.0)
- added R1: 100kΩ, Resistor_SMD:R_0603_1608Metric, F.Cu at (168.9, 94.3)
- added R17: 4.7k, Resistor_SMD:R_0603_1608Metric, F.Cu at (176.9, 86.8)
- added R18: 4.7k, Resistor_SMD:R_0603_1608Metric, F.Cu at (176.9, 89.3)
- added R19: 0, Resistor_SMD:R_1206_3216Metric, F.Cu at (151.2, 106.4)
- added R2: 100kΩ, Resistor_SMD:R_0603_1608Metric, F.Cu at (172.9, 79.3)
- added R20: 0, Resistor_SMD:R_1206_3216Metric, F.Cu at (151.2, 109.7)
- added R21: 0, Resistor_SMD:R_1206_3216Metric, F.Cu at (151.2, 113.0)
- added R23: 0, Resistor_SMD:R_1206_3216Metric, F.Cu at (151.2, 116.3)
- added U6: TPS62133, Package_DFN_QFN:VQFN-16-1EP_3x3mm_P0.5mm_EP1.68x1.68mm_ThermalVias, F.Cu at (177.0, 116.3)
- U4: value TPS62130A -> TPS62132
- moved C4 85.3 mm to (164.9, 86.8), turned to 0 degrees
- moved J2 82.9 mm to (151.9, 81.4), turned to 0 degrees
- moved H2 80.6 mm to (66.7, 118.4)
- moved H1 66.1 mm to (66.7, 75.3)
- moved U4 55.6 mm to (176.2, 111.2)
- moved J6 52.3 mm to (135.5, 89.2)
- moved J5 38.5 mm to (135.5, 81.4)
- moved R14 35.7 mm to (176.9, 79.3)
- moved R15 35.7 mm to (176.9, 81.8)
- moved R5 35.7 mm to (172.9, 81.8)
- moved SW1 32.1 mm to (156.3, 103.7)
- moved SW2 32.1 mm to (160.9, 103.7)
- moved SW3 32.1 mm to (165.5, 103.7)
- moved H4 29.1 mm to (121.9, 118.3)
- moved C15 26.3 mm to (168.9, 91.8)
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Connections:
- net +6.2V renamed Net-(U4-EN)
- C15 pad 2: +3v3 -> +3V3
- D10 pad 2: +3V3 -> Net-(D10-A)
- J5 pad 1: +5V -> Net-(J11-Pin_1)
- J6 pad 1: +5V -> Net-(J11-Pin_1)
- J7 pad 1: +5V -> Net-(J11-Pin_1)
- R14 pad 2: +3.3V -> +3V3
- R15 pad 2: +3.3V -> +3V3
- R22 pad 1: GND -> Net-(J10-CC2)
- R22 pad 2: Net-(J3-CC2) -> GND
- SW3 pad 2: +3.3V -> +3V3
- U1 pad 5: V_{USB-C} -> V_USB
- U2 pad 12: unconnected-(U2-IO8-Pad12) -> /OLED_SDA
- U2 pad 17: unconnected-(U2-IO9-Pad17) -> /PWR_Enable
- U2 pad 7: unconnected-(U2-IO7-Pad7) -> /OLED_SCL
- U3 pad 3: +3v3 -> +3V3
- U4 pad 14: +5V -> +3V3
- U4 pad 15: Net-(U4-GND-Pad15) -> GND
- U4 pad 16: Net-(U4-GND-Pad15) -> GND
- U4 pad 17: Net-(U4-GND-Pad15) -> GND
- U4 pad 4: unconnected-(U4-PG-Pad4) -> Net-(U4-PG)
- U4 pad 5: unconnected-(U4-FB-Pad5) -> GND
- U4 pad 6: Net-(U4-GND-Pad15) -> GND
- U4 pad 7: unconnected-(U4-FSW-Pad7) -> GND
- U4 pad 8: unconnected-(U4-DEF-Pad8) -> GND
- U4 pad 9: unconnected-(U4-SS/TR-Pad9) -> Net-(U4-SS/TR)
Routing:
- net +3V3: track 16.6 -> 0.00 mm
- net /Mother_{TX}: track 15.6 -> 0.00 mm, vias 2 -> 0
- net /Mother_{RX}: track 15.1 -> 0.00 mm
- net (no net): track 5.08 -> 0.00 mm
- added copper zone on F.Cu, net +3V3
- removed copper zone on F.Cu, net +5V
Other:
- board size 60.4 x 48.6 mm -> 62.4 x 50.3 mm

Commit message: <UPDATE> Oliver Review Ver
Parts:
- removed R16: 10k, Resistor_SMD:R_0603_1608Metric
- removed SW3: SW_Push, Connector_PinHeader_2.54mm:PinHeader_1x02_P2.54mm_Vertical
- J8: footprint Connector_JST:JST_XH_B2B-XH-A_1x02_P2.50mm_Vertical -> Connector_PinHeader_2.54mm:PinHeader_1x02_P2.54mm_Vertical
- moved H3 117.3 mm to (18.4, 20.1)
- moved J10 116.6 mm to (68.1, 84.5)
- moved H2 115.8 mm to (14.3, 15.1)
- moved R17 105.4 mm to (71.6, 92.5), turned to 90 degrees
- moved R18 105.4 mm to (71.7, 95.6), turned to 90 degrees
- moved R13 103.4 mm to (70.8, 77.9), turned to 180 degrees
- moved R22 103.2 mm to (73.7, 91.3), turned to -90 degrees
- moved R2 96.9 mm to (77.5, 96.2), turned to 180 degrees
- moved U4 95.7 mm to (81.8, 95.0)
- moved R12 95.1 mm to (78.3, 81.9)
- moved R8 93.4 mm to (80.0, 79.6), turned to 180 degrees
- moved R7 93.3 mm to (80.0, 77.7), turned to 180 degrees
- moved C8 92.1 mm to (77.6, 91.4), turned to -90 degrees
- moved U1 88.1 mm to (78.3, 84.7)
- moved J4 85.8 mm to (66.9, 101.2), turned to 90 degrees
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Connections:
- C3 pad 2: Net-(U6-VOS) -> +5V
- J2 pad 3: /Mother_{TX} -> /Mother_{RX}
- J2 pad 4: /Mother_{RX} -> /Mother_{TX}
- L1 pad 2: Net-(U6-VOS) -> +5V
- R1 pad 2: Net-(U6-VOS) -> +5V
- R17 pad 1: /OLED_SDA -> /OLED_SCL
- R18 pad 1: /OLED_SCL -> /OLED_SDA
- U2 pad 12: /OLED_SDA -> unconnected-(U2-IO8-Pad12)
- U2 pad 16: /GPIO_{6} -> unconnected-(U2-IO46-Pad16)
- U2 pad 17: /PWR_Enable -> unconnected-(U2-IO9-Pad17)
- U2 pad 24: /GPIO_{8} -> unconnected-(U2-IO47-Pad24)
- U2 pad 25: /GPIO_{7} -> unconnected-(U2-IO48-Pad25)
- U2 pad 26: /GPIO_{5} -> /PWR_Enable
- U2 pad 28: unconnected-(U2-IO35-Pad28) -> /GPIO_{1}
- U2 pad 29: unconnected-(U2-IO36-Pad29) -> /GPIO_{2}
- U2 pad 30: unconnected-(U2-IO37-Pad30) -> /GPIO_{3}
- U2 pad 31: unconnected-(U2-IO38-Pad31) -> /GPIO_{4}
- U2 pad 32: /GPIO_{1} -> /GPIO_{5}
- U2 pad 33: /GPIO_{2} -> /GPIO_{6}
- U2 pad 34: /GPIO_{3} -> /GPIO_{7}
- U2 pad 35: /GPIO_{4} -> /GPIO_{8}
- U2 pad 38: /Safe Boot -> unconnected-(U2-IO2-Pad38)
- U2 pad 4: unconnected-(U2-IO4-Pad4) -> /LED_{1}
- U2 pad 5: /LED_{1} -> /LED_{2}
- U2 pad 6: /LED_{2} -> /OLED_SCL
- U2 pad 7: /OLED_SCL -> /OLED_SDA
- U6 pad 14: Net-(U6-VOS) -> +5V
Routing:
- net GND: track 0.00 -> 80.0 mm, vias 0 -> 24
- net /Boot Mode: track 0.00 -> 71.1 mm, vias 0 -> 2
- net /EN: track 0.00 -> 69.1 mm, vias 0 -> 2
- net Net-(J11-Pin_1): track 0.00 -> 66.3 mm
- net +6V2: track 0.00 -> 30.3 mm, vias 0 -> 2
- net /OLED_SDA: track 0.00 -> 28.4 mm, vias 0 -> 2
- net /OLED_SCL: track 0.00 -> 27.8 mm, vias 0 -> 2
- net V_USB: track 0.00 -> 26.5 mm
- net /Mother_{TX}: track 0.00 -> 22.7 mm, vias 0 -> 1
- net /Mother_{RX}: track 0.00 -> 20.8 mm, vias 0 -> 1
- net +5V: track 0.00 -> 17.4 mm
- net /GPIO_{2}: track 0.00 -> 15.7 mm
- net /GPIO_{1}: track 0.00 -> 14.0 mm
- net Net-(F1-Pad2): track 0.00 -> 13.9 mm
- net Net-(U4-EN): track 0.00 -> 12.9 mm
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Other:
- board size 62.4 x 50.3 mm -> 62.4 x 33.9 mm
