File: hardware/rev2/TyphoonMotherboard_rev1 KiCad.kicad_pcb (KiCad board)
At the start: 2 copper layers, 62.4 x 33.9 mm, 57 parts, among them J1 Conn_02x04_Odd_Even, J10 USB_C_Receptacle_USB2.0_16P, J11 Conn_01x02_Pin, J2 Conn_01x04_Pin, J4 Conn_01x04_Pin, J5 Conn_01x02_Pin, J6 Conn_01x02_Pin, J7 Conn_01x04_Pin, J8 Conn_01x02_Pin, J9 Conn_01x02_Pin, SW1 SW_Push, SW2 SW_Push, U1 USBLC6-2SC6, U2 ESP32-S3-WROOM-1, U3 SN65HVD233, U4 TPS62132, U6 TPS62133

Commit message: <UPDATE> Ordered Board
Parts:
- removed C10: 3.3nF, Capacitor_SMD:C_0603_1608Metric
- removed C6: 4.7n, Capacitor_SMD:C_0603_1608Metric
- removed C7: 10uF, Capacitor_SMD:C_0603_1608Metric
- removed D4: LED, LED_SMD:LED_0805_2012Metric
- removed F1: Polyfuse, Fuse:Fuse_1206_3216Metric
- removed L2: 2.2uH, Inductor_SMD:L_0805_2012Metric
- removed R2: 100kΩ, Resistor_SMD:R_0603_1608Metric
- removed R6: 60, Resistor_SMD:R_0603_1608Metric
- removed R8: 320, Resistor_SMD:R_0603_1608Metric
- C11: value 0.1uF -> 1uF
- C12: value 0.1uF -> 4.7u
- C8: value 22uF -> 4.7u
- R5: value 60 -> 120
- SW1, SW2: footprint Connector_PinHeader_2.54mm:PinHeader_1x02_P2.54mm_Vertical -> SWITCH_MOTHERBOARD:SMT_FS
- U4: value TPS62132 -> MCP1804x-3302xDB; footprint Package_DFN_QFN:VQFN-16-1EP_3x3mm_P0.5mm_EP1.68x1.68mm_ThermalVias -> Package_TO_SOT_SMD:SOT-223-3_TabPin2
- moved R15 20.9 mm to (115.1, 74.9), turned to -90 degrees
- moved SW1 15.0 mm to (121.3, 89.2)
- moved J6 10.5 mm to (115.5, 101.9), turned to 180 degrees
- moved SW2 7.73 mm to (121.4, 95.5)
- moved C8 6.93 mm to (84.3, 93.3)
- moved R14 4.30 mm to (116.3, 96.3), turned to 90 degrees
- moved R20 3.98 mm to (76.2, 88.0), turned to 135 degrees
- moved U4 2.96 mm to (79.0, 94.1), turned to 180 degrees
- moved R5 2.11 mm to (116.8, 76.7)
- moved H4 1.41 mm to (122.5, 102.6)
- moved C12 1.38 mm to (84.3, 96.3)
- moved J11 1.14 mm to (106.9, 101.9)
- moved J5 1.07 mm to (98.4, 101.9)
- moved J9 0.83 mm to (89.8, 102.0)
- moved J7 0.78 mm to (120.9, 82.9)
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Connections:
- C12 pad 1: GND -> +3V3
- C12 pad 2: Net-(U4-EN) -> GND
- C8 pad 1: GND -> Net-(U4-IN)
- C8 pad 2: +3V3 -> GND
- J10 pad A4: Net-(F1-Pad2) -> V_USB
- J10 pad A9: Net-(F1-Pad2) -> V_USB
- J10 pad B4: Net-(F1-Pad2) -> V_USB
- J10 pad B9: Net-(F1-Pad2) -> V_USB
- R19 pad 1: Net-(U4-EN) -> Net-(U4-IN)
- R20 pad 1: Net-(U4-EN) -> Net-(U4-IN)
- R5 pad 2: Net-(C6-Pad1) -> /CAN-
- U2 pad 5: /LED_{2} -> unconnected-(U2-IO5-Pad5)
- U4 pad 1: Net-(L2-Pad1) -> +3V3
- U4 pad 2: Net-(L2-Pad1) -> GND
- U4 pad 3: Net-(L2-Pad1) -> Net-(U4-IN)
Routing:
- net V_USB: track 26.5 -> 41.0 mm
- net /Boot Mode: track 71.1 -> 57.0 mm
- net Net-(F1-Pad2): track 13.9 -> 0.00 mm
- net Net-(U4-IN): track 0.00 -> 13.1 mm
- net Net-(U4-EN): track 12.9 -> 0.00 mm
- net Net-(L2-Pad1): track 7.60 -> 0.00 mm
- net Net-(J11-Pin_1): track 66.3 -> 59.1 mm
- net Net-(U4-SS/TR): track 7.18 -> 0.00 mm
- net /LED_{2}: track 6.14 -> 0.00 mm
- net GND: track 80.0 -> 74.2 mm, vias 24 -> 20
- net Net-(C6-Pad1): track 3.47 -> 0.00 mm
- net /EN: track 69.1 -> 66.7 mm
- net Net-(U4-PG): track 2.25 -> 0.00 mm
- net Net-(D4-A): track 2.12 -> 0.00 mm
- net +3V3: track 7.24 -> 9.35 mm, vias 1 -> 0
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