File: hardware/rev2/TyphoonMotherboard_rev1 KiCad.kicad_sch (KiCad schematic)
At the start: 57 parts, among them J1 Conn_02x04_Odd_Even, J10 USB_C_Receptacle_USB2.0_16P, J11 Conn_01x02_Pin, J2 Conn_01x04_Pin, J4 Conn_01x04_Pin, J5 Conn_01x02_Pin, J6 Conn_01x02_Pin, J7 Conn_01x04_Pin, J8 Conn_01x02_Pin, J9 Conn_01x02_Pin, SW1 SW_Push, SW2 SW_Push, U1 USBLC6-2SC6, U2 ESP32-S3-WROOM-1, U3 SN65HVD233, U4 TPS62132, U6 TPS62133

Commit message: <UPDATE> Ordered Board
Parts:
- removed C10: 3.3nF, Capacitor_SMD:C_0603_1608Metric, symbol Device:C
- removed C12: 0.1uF, Capacitor_SMD:C_0603_1608Metric, symbol Device:C
- removed C6: 4.7n, Capacitor_SMD:C_0603_1608Metric, symbol Device:C
- removed C7: 10uF, Capacitor_SMD:C_0603_1608Metric, symbol Device:C
- removed C8: 22uF, Capacitor_SMD:C_0603_1608Metric, symbol Device:C
- removed D4: LED, LED_SMD:LED_0805_2012Metric, symbol Device:LED
- removed F1: Polyfuse, Fuse:Fuse_1206_3216Metric, symbol Device:Polyfuse
- removed L2: 2.2uH, Inductor_SMD:L_0805_2012Metric, symbol Device:L
- removed R2: 100kΩ, Resistor_SMD:R_0603_1608Metric, symbol Device:R
- removed R6: 60, Resistor_SMD:R_0603_1608Metric, symbol Device:R
- removed R8: 320, Resistor_SMD:R_0603_1608Metric, symbol Device:R
- removed U4: TPS62132, Package_DFN_QFN:VQFN-16-1EP_3x3mm_P0.5mm_EP1.68x1.68mm_ThermalVias, symbol Regulator_Switching:TPS62132
- added C12, C8: 4.7u, Capacitor_SMD:C_0603_1608Metric, symbol Device:C_Small
- added U4: MCP1804x-3302xDB, Package_TO_SOT_SMD:SOT-223-3_TabPin2, symbol Regulator_Linear:MCP1804x-3302xDB
- C11: value 0.1uF -> 1uF
- R13: value 330 -> 320
- R5: value 60 -> 120
- SW1, SW2: footprint (none) -> SWITCH_MOTHERBOARD:SMT_FS
Connections:
- net +3V3: now also C12.1, U4.1 (OUT)
- net CAN-: now also R5.2
- net GND: now also C12.2, C8.2, U4.2 (GND)
- net V_USB: now also J10.A4 (VBUS), J10.A9 (VBUS), J10.B4 (VBUS), J10.B9 (VBUS)
- net at R19.1, R20.1: now also C8.1, U4.3 (IN)
- net LED_{2}: no longer names the net of U2.5 (IO5)
- no-connect marks 18 -> 19
Other:
- note added: "3V3 LDO"
- note removed: "3V3 Buck Converter"
- moved on the sheet: R5
